File: dawcontrol.kicad_sch (KiCad schematic)
At the start: 5 parts, among them U1 STM32L552ZETxQ

Commit message: Add kicad librarys
Parts:
- added D5, D6, D7, D8: WS2812B, LED_SMD:LED_WS2812B_PLCC4_5.0x5.0mm_P3.2mm, symbol LED:WS2812B
- added M1, M2, M3, M4, M5, M6, M7, M8: Motor_DC, symbol Motor:Motor_DC
- added RV1, RV2, RV3, RV4, RV5, RV6, RV7, RV8: R_Potentiometer, symbol Device:R_Potentiometer
- added SW1, SW2, SW3, SW4, SW5, SW6, SW7, SW8: RotaryEncoder, symbol Device:RotaryEncoder
- added U10, U16, U17, U23, U24, U30, U31, U37, U38, U44, U45, U51, U52, U7, U8, U9: ER_OLEDM0.91_1x-I2C, Display:ER_OLEDM0.91_1x-I2C, symbol Display_Graphic:ER_OLEDM0.91_1x-I2C
- added U11, U12, U13, U14, U15, U18, U19, U2, U20, U21, U22, U25, U26, U27, U28, U29, U3, U32, U33, U34, U35, U36, U39, U4, U40, U41, U42, U43, U46, U47, U48, U49, U5, U50, U53, U54, U55, U56, U57, U6: CherryMX_LTST-A683CEGBW, symbol CherryMX:CherryMX_LTST-A683CEGBW
- added U58: 74HC165, symbol 74xx:74HC165
- added U59: STM32G0B0KETx, Package_QFP:LQFP-32_7x7mm_P0.8mm, symbol MCU_ST_STM32G0:STM32G0B0KETx
Connections:
- net +5V: no longer D1.1 (VDD), D2.1 (VDD), D3.1 (VDD), D4.1 (VDD)
- net D11: no longer D1.4 (DIN)
- net GND: no longer D1.3 (VSS), D2.3 (VSS), D3.3 (VSS), D4.3 (VSS)
- net at D3.2 (DOUT): no longer D4.4 (DIN)
- net at D3.4 (DIN): no longer D2.2 (DOUT)
- net at D1.2 (DOUT): no longer D2.4 (DIN)
Other:
- moved on the sheet: U1

Commit message: Add button section for schematic
Parts:
- removed D1, D2, D3, D4, D5, D6, D7, D8: WS2812B, LED_SMD:LED_WS2812B_PLCC4_5.0x5.0mm_P3.2mm, symbol LED:WS2812B
- removed M1, M2, M3, M4, M5, M6, M7, M8: Motor_DC, symbol Motor:Motor_DC
- removed RV1, RV2, RV3, RV4, RV5, RV6, RV7, RV8: R_Potentiometer, symbol Device:R_Potentiometer
- removed SW3, SW4, SW5, SW6, SW7, SW8: RotaryEncoder, symbol Device:RotaryEncoder
- removed U11, U12, U13, U14, U15, U18, U19, U2, U20, U21, U22, U25, U26, U27, U28, U29, U32, U33, U34, U35, U36, U39, U40, U41, U42, U43, U46, U47, U48, U49, U50, U53, U54, U55, U56, U57, U6: CherryMX_LTST-A683CEGBW, symbol CherryMX:CherryMX_LTST-A683CEGBW
- removed U16, U17, U23, U24, U30, U31, U37, U38, U44, U45, U51, U52: ER_OLEDM0.91_1x-I2C, Display:ER_OLEDM0.91_1x-I2C, symbol Display_Graphic:ER_OLEDM0.91_1x-I2C
- removed U58: 74HC165, symbol 74xx:74HC165
- removed U59: STM32G0B0KETx, Package_QFP:LQFP-32_7x7mm_P0.8mm, symbol MCU_ST_STM32G0:STM32G0B0KETx
- added C1, C2, C3, C4, C5, C6, C7, C8: 0.1uF, symbol Device:C
- added CH1-Select, CH2-Mute, CH2-Record/Monitor, CH2-Select, CH2-Solo: CherryMX_LTST-A683CEGBW, symbol CherryMX:CherryMX_LTST-A683CEGBW
- added R1, R2, R3, R4, R5, R6, R7, R8: R, symbol Device:R
- added R10, R11, R12, R13, R14, R15, R16, R9: 10kΩ, symbol Device:R
- added U2: 74HC165, symbol 74xx:74HC165
- added U4, U5: ALPS_RSA0N11M9A0J, symbol vitalis_personal_lib:ALPS_RSA0N11M9A0J
- renumbered U5 to CH1-Mute, U3 to CH1-Record/Monitor, U4 to CH1-Solo
Connections:
- net GND: now also CH1-Mute.1, CH1-Mute.3 (VSS), CH1-Record/Monitor.1, CH1-Record/Monitor.3 (VSS), CH1-Solo.1, CH1-Solo.3 (VSS), C1.2, C2.2, C3.2, C4.2, C5.2, C6.2, C7.2, C8.2, CH1-Select.1, CH1-Select.3 (VSS), CH2-Mute.1, CH2-Mute.3 (VSS), CH2-Record/Monitor.1, CH2-Record/Monitor.3 (VSS), CH2-Select.1, CH2-Select.3 (VSS), CH2-Solo.1, CH2-Solo.3 (VSS), U2.15 (~{CE}), U2.8 (GND)
- net HC_D3: now reaches CH1-Record/Monitor.2
- net HC_D3: now also R12.2, U2.14 (D3)
- net at CH1-Record/Monitor.4 (DIN): now also CH1-Solo.5 (DOUT)
- net led_chain: now reaches CH1-Record/Monitor.6 (VDD)
- net led_chain: now also C3.1, CH2-Select.4 (DIN), R3.2
- net HC_D2: now reaches CH1-Solo.2
- net HC_D2: now also R11.2, U2.13 (D2)
- net at CH1-Solo.4 (DIN): now also CH1-Mute.5 (DOUT)
- net at CH1-Solo.6 (VDD): now also C2.1, R2.2
- net HC_D1: now reaches CH1-Mute.2
- net HC_D1: now also R10.2, U2.12 (D1)
- net at CH1-Mute.4 (DIN): now also CH1-Select.5 (DOUT)
- net at CH1-Mute.6 (VDD): now also C1.1, R1.2
- new net: C6.1, CH2-Mute.6 (VDD), R6.2
- new net: C7.1, CH2-Solo.6 (VDD), R7.2
- new net: C4.1, CH1-Select.6 (VDD), R4.2
- new net: CH2-Record/Monitor.4 (DIN), CH2-Solo.5 (DOUT)
- new net: C8.1, CH2-Record/Monitor.6 (VDD), R8.2
- new net: C5.1, CH2-Select.6 (VDD), R5.2
- new net: CH2-Mute.4 (DIN), CH2-Select.5 (DOUT)
- new net: CH2-Mute.5 (DOUT), CH2-Solo.4 (DIN)
- new net +5.5V: R1.1, R10.1, R11.1, R12.1, R13.1, R14.1, R15.1, R16.1, R2.1, R3.1, R4.1, R5.1, R6.1, R7.1, R8.1, R9.1, U2.16 (VCC)
- new net HC_D0: CH1-Select.2, R9.2, U2.11 (D0)
- new net HC_D4: CH2-Select.2, R13.2, U2.3 (D4)
- new net HC_D5: CH2-Mute.2, R14.2, U2.4 (D5)
- new net HC_D6: CH2-Solo.2, R15.2, U2.5 (D6)
- new net HC_D7: CH2-Record/Monitor.2, R16.2, U2.6 (D7)
Other:
- note added: "Button Section"
- note added: "Pull PL low to capture the register. Then readout with applying clock to CP."
- moved on the sheet: CH1-Mute, CH1-Record/Monitor, CH1-Solo

Commit message: Add first controller selection
Parts:
- removed C1, C2, C3, C4, C5, C6, C7, C8: 0.1uF, symbol Device:C
- removed CH1-Mute, CH1-Record/Monitor, CH1-Select, CH1-Solo, CH2-Mute, CH2-Record/Monitor, CH2-Select, CH2-Solo: CherryMX_LTST-A683CEGBW, symbol CherryMX:CherryMX_LTST-A683CEGBW
- removed R1, R2, R3, R4, R5, R6, R7, R8: R, symbol Device:R
- added CH1-Mute, CH1-Record/Monitor, CH1-Select, CH1-Solo, CH2-Mute, CH2-Record/Monitor, CH2-Select, CH2-Solo: CherryMX_SK6812MINI-E, symbol vitalis_personal_lib:CherryMX_SK6812MINI-E
- added R17, R18: 10kΩ, symbol Device:R
- added U3: STM32G0B1KETx, Package_QFP:LQFP-32_7x7mm_P0.8mm, symbol MCU_ST_STM32G0:STM32G0B1KETx
- added U6: TB6612FNG, Package_SO:SSOP-24_5.3x8.2mm_P0.65mm, symbol Driver_Motor:TB6612FNG
Connections:
- net +5.5V: now also CH1-Mute.2 (VDD), CH1-Record/Monitor.2 (VDD), CH1-Select.2 (VDD), CH1-Solo.2 (VDD), CH2-Mute.2 (VDD), CH2-Record/Monitor.2 (VDD), CH2-Select.2 (VDD), CH2-Solo.2 (VDD)
- net +5V: now also U4.3 (100%), U5.3 (100%)
- net GND: now also U4.1 (0%), U5.1 (0%), CH1-Mute.1 (DIN), CH1-Mute.4 (GND), CH1-Record/Monitor.1 (DIN), CH1-Record/Monitor.4 (GND), CH1-Select.1 (DIN), CH1-Select.4 (GND), CH1-Solo.1 (DIN), CH1-Solo.4 (GND), CH2-Mute.1 (DIN), CH2-Mute.4 (GND), CH2-Record/Monitor.1 (DIN), CH2-Record/Monitor.4 (GND), CH2-Select.1 (DIN), CH2-Solo.1 (DIN), CH2-Solo.4 (GND)
- net HC_D0: now also CH1-Select.2 (VDD)
- net HC_D1: now also CH1-Mute.2 (VDD)
- net HC_D2: now also CH1-Solo.2 (VDD)
- net HC_D3: now also CH1-Record/Monitor.2 (VDD)
- net HC_D4: now also CH2-Select.2 (VDD)
- net HC_D5: now also CH2-Mute.2 (VDD)
- net HC_D6: now also CH2-Solo.2 (VDD)
- net HC_D7: now also CH2-Record/Monitor.2 (VDD)
- net button_register_capture: now reaches U2.1 (~{PL})
- net button_register_capture: now also U3.29 (PB5)
- net button_register_clock: now reaches U2.2 (CP)
- net button_register_clock: now also U3.27 (PB3)
- net button_register_readout: now reaches U2.9 (Q7)
- net button_register_readout: now also U3.28 (PB4)
- new net: CH2-Mute.1 (DIN), CH2-Select.3 (DOUT)
- new net: CH2-Mute.3 (DOUT), CH2-Solo.1 (DIN)
- new net: CH1-Mute.1 (DIN), CH1-Select.3 (DOUT)
- new net: CH1-Mute.3 (DOUT), CH1-Solo.1 (DIN)
- new net: CH2-Record/Monitor.3 (DOUT), R18.1
- new net: CH2-Record/Monitor.1 (DIN), CH2-Solo.3 (DOUT)
- new net: CH1-Record/Monitor.1 (DIN), CH1-Solo.3 (DOUT)
- new net: CH1-Select.1 (DIN), R17.2
- new net: U6.1 (AO1), U6.2 (AO1)
- new net: U6.10 (PGND2), U6.9 (PGND2)
- new net: U6.11 (BO1), U6.12 (BO1)
- new net: U6.3 (PGND1), U6.4 (PGND1)
- new net: U6.5 (AO2), U6.6 (AO2)
- new net: U6.7 (BO2), U6.8 (BO2)
- new net: CH1-Record/Monitor.3 (DOUT), CH2-Select.4 (GND)
- new net led_in: R17.1, U3.32 (PB8)
Other:
- moved on the sheet: R10, R11, R12, R13, R14, R15, R16, R9, U2, U4, U5

Commit message: Fader section
Parts:
- added C1, C4: 0.1uF, symbol Device:C
- added C2, C3: 10uF, symbol Device:C_Polarized
Connections:
- net +5V: now also U6.20 (VCC), C3.1, C4.2; no longer U4.3 (100%), U5.3 (100%)
- net GND: now also U6.10 (PGND2), U6.18 (GND), U6.3 (PGND1), U6.4 (PGND1), U6.9 (PGND2), C1.1, C2.2, C3.2, C4.1
- net fader_1_whiper: now reaches U4.2 (Wiper)
- net at U4.A: now also U6.5 (AO2), U6.6 (AO2)
- net at U4.B: now also U6.1 (AO1), U6.2 (AO1)
- net fader_1_sense: now reaches U4.T (Lever)
- net at U6.11 (BO1), U6.12 (BO1): now also U5.B
- net +4V5 to +13V5: now reaches U6.13 (VM2)
- net +4V5 to +13V5: now also U6.14 (VM3), U6.24 (VM1), C1.2, C2.1
- net fader_2_drive_speed: now reaches U6.15 (PWMB)
- net fader_2_drive_direction_2: now reaches U6.16 (BIN2)
- net fader_2_drive_direction_1: now reaches U6.17 (BIN1)
- net fader_drive_stby: now reaches U6.19 (STBY)
- net fader_1_drive_direction_1: now reaches U6.21 (AIN1)
- net fader_1_drive_direction_2: now reaches U6.22 (AIN2)
- net fader_1_drive_speed: now reaches U6.23 (PWMA)
- net at U6.7 (BO2), U6.8 (BO2): now also U5.A
- net fader_2_whiper: now reaches U5.2 (Wiper)
- net fader_2_sense: now reaches U5.T (Lever)
- new net +3V3: U4.3 (100%), U5.3 (100%)
Other:
- note added: "Fader Section"
- note added: "Motor stby musst be pulled HIGH to drive the motors. Condensers for noise absorption (C1, C2, C3, and C4) should be connected as close as possible to the IC."
- moved on the sheet: U4, U5
